File: iot-wifi-uno-hw.sch (KiCad schematic (older format))
At the start: 61 parts, among them CON1 BARREL_JACK, P1 CONN_01X08, P2 CONN_01X08, P3 CONN_01X06, P4 CONN_01X10, P5 CONN_01X04, Q1 Q_NPN_BEC, Q2 Q_NPN_BEC, U1 usb_mini_b, U2 MCP16311-MNY, U3 CH340G, U4 ESP-12E, U5 MCP6001R, U6 BD00GA5WEFJ, U7 IRLM6402, X1 CRYSTAL_ABM3C

Commit message: Fix error button & modify pwr for CH340G 5v to 3.3V (#15)
* fix via beetwen U3 & R16

* Delete fp-lib-table

* deleted iot-wifi-uno-hw-cache.lib

* Fix crystall of CH340G

* modify some track

* Modify footprint MCP16311, add zener to ADC, fix footprint 2 transistor

* Fix PCB diode zenner right

* Completed PCB & Boom list & Update Gerber file

* update README file

* Modify Bom lish to Markdown Tables

* Fix Zone at module wifi esp-12

* update picture PCB

* Modify Zone module ESP-12

* fix transistor to 1b 2e 3c on datasheet MMBT8050

* update picture PCB & SCH

* Fix Via & update assets

* update picture SVG file PCB

* Add file SVG pinout & picture pinout

* update pinout file

* change IC CH340G to PL2303HXD

* setup new PCB

* fix error button & modify CH340G 5V to 3.3V, Update PCB

* update gerber file
Parts:
- removed D5: ZENER_3.3V, ESP8266:SOD-80, symbol ZENER_Small
- removed GPIO1: GPIO0, ESP8266:Tact_Switch_TS6X3.6, symbol SW_PUSH_Small_Horizontal
- removed L1: 22uH, Choke_SMD:Choke_SMD_Wuerth-WE-PD2-Typ-MS, symbol INDUCTOR_Small
- removed RST1: REST, ESP8266:Tact_Switch_TS6X3.6, symbol SW_PUSH_Small_Horizontal
- added D5: ZENER_3.3V, ESP8266:SOD-80, symbol D_Schottky_Small
- added L1: 22uH, Choke_SMD:Choke_SMD_Wuerth-WE-PD2-Typ-MS, symbol L_Small
- added SW1: RST, ESP8266:Tact_Switch_TS6X3.6, symbol SW_PUSH
- added SW2: GPIO0, ESP8266:Tact_Switch_TS6X3.6, symbol SW_PUSH
- Q1, Q2: value Q_NPN_BEC -> MMBT8050LT1G_BEC
Connections:
- wire segments 281 -> 230
Other:
- moved on the sheet: C10, C11, C12, C3, C4, C6, C7, C9, CON1, D1, Q1, Q2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

Commit message: feature/power (#16)
* ?

* edited pcb

* pcb layout hoan chỉnh

* pcb layout hoàn chỉnh

* pcb layout hoàn chỉnh

* Update .gitignore

* pcb hoàn chỉnh, add 3d, khung

* pcb hoàn chỉnh, add 3d, khung

* Update .gitignore

* PCB layout hoàn chỉnh, sửa khung, sửa 3d hoàn chỉnh

* Update .gitignore

* PCB layout hoàn chỉnh, sửa khung, sửa 3d hoàn chỉnh, sửa lỗi thư viện

* pcb layout hoàn chỉnh, sửa lỗi vị trí linh kiện, schematic

* sửa schematic

* PCB layout sửa xong

* pcb hoàn chỉnh, sửa lỗi 3d, schematic, tên footprint
Parts:
- removed C10, C11: 10uF/25V, ESP8266:C_1210, symbol C_Small
- removed C7: 1uF, ESP8266:C_0603, symbol C_Small
- removed C9: 100nF, ESP8266:C_0603, symbol C_Small
- removed D1: SS24, ESP8266:do214aa-g, symbol D_Schottky_Small
- removed L1: 22uH, Choke_SMD:Choke_SMD_Wuerth-WE-PD2-Typ-MS, symbol L_Small
- removed P1, P2: CONN_01X08, Pin_Headers:Pin_Header_Straight_1x08, symbol CONN_01X08
- removed P3: CONN_01X06, Pin_Headers:Pin_Header_Straight_1x06, symbol CONN_01X06
- removed P4: CONN_01X10, Pin_Headers:Pin_Header_Straight_1x10, symbol CONN_01X10
- removed P5: CONN_01X04, Pin_Headers:Pin_Header_Straight_1x04, symbol CONN_01X04
- removed R20: 3K/1%, ESP8266:R_0603, symbol R_Small
- removed R21: 1K/1%, ESP8266:R_0603, symbol R_Small
- removed R8: 52.5K, ESP8266:R_0603, symbol R_Small
- removed R9: 10k, ESP8266:R_0603, symbol R_Small
- removed U2: MCP16311-MNY, Housings_SSOP:MSOP-8_3x3mm_Pitch0.65mm, symbol MCP16311-MNY
- removed U6: BD00GA5WEFJ, ESP8266:HTSOP-J8, symbol BD00GA5WEFJ
- added D1: SCHOTTKY, ESP8266:do214aa-g, symbol SCHOTTKY
- added S1: ESP-UNO, ESP8266:shield-uno, symbol ESP-UNO-RESCUE-iot-wifi-uno-hw-RESCUE-iot-wifi-uno-hw
- added U2: AMS117-5.0, TO_SOT_Packages_SMD:SOT-223-3Lead_TabPin2, symbol LD1117S12TR_SOT223
- added U6: AMS1117-3.3, TO_SOT_Packages_SMD:SOT-223-3Lead_TabPin2, symbol LD1117S12TR_SOT223
- C3, C4: value 10uF/50V -> 1uF/25V
- CON1: symbol BARREL_JACK -> Barrel_Jack
Connections:
- wire segments 230 -> 198
- no-connect marks 18 -> 14
Other:
- note removed: "A1\n"
- note removed: "A2\n"
- note removed: "ADC0"
- note removed: "HEADER GPIO"
- note removed: "HEADER_OLED"
- note removed: "MISO"
- note removed: "MOSI\n"
- note removed: "SCK"
- note removed: "SCL"
- note removed: "SDA"
- note removed: "SDA\n"
- note removed: "SS"
- moved on the sheet: C12, C13, C14, C15, C6, D2, D3, D4, D5, Q1, Q2, R10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
